File: RP2040_motor.kicad_pcb (KiCad board)
At the start: 4 copper layers, 114.1 x 83.2 mm, 438 parts, among them J1 CPU1 USB, J10 AUX GPIO 1, J11 CAN2 PLUG, J12 Conn_01x06, J13 ADC AUX 2, J14 AUX GPIO 2, J15 AUX Encoder, J17 CAN Output, J19 Conn_01x03, J2 CAN Input, J20 Conn_01x03, J21 Power Input, J3 Encoder 1, J4 Encoder 2, J5 Conn_01x06, J6 CPU2 USB, J7 Conn_01x02, J9 ADC AUX 1, Q1 Q_PNP_BEC, Q2 Q_PNP_BEC, Q3 Q_PNP_BEC, Q4 Q_PNP_BEC, Q5 Q_PNP_BEC, Q6 Q_PNP_BEC, Q7 Q_NMOS_GSD, SW1 SW_MEC_5G, SW2 SW_MEC_5G, SW3 CONFIG SWITCH, U1 EG2131, U10 TXS0101DCKR, U11 TLV1117LV33DCYR, U12 W25Q128JVSIQ, U13 W25Q128JVSIQ, U14 INA193, U15 RP2040, U16 ADC081S021CISD/NOPB, U17 isolator, U18 MCP2515-xSO, U19 RP2040, U2 EG2131, U20 INA193, U21 INA193, U22 INA193, U23 SN74LVC1G07QDCKTQ1, U24 MT2492, U25 NCP1117-5_SOT223, U26 ADC081S021CISD/NOPB, U27 USBLC6-2P6, U28 USBLC6-2P6, U29 USBLC6-4SC6, U3 USBLC6-4SC6, U30 USBLC6-4SC6, U31 USBLC6-4SC6, U32 TLV1117LV33DCYR, U33 TX4139, U34 LTV-208, U35 INA193, U36 INA826, U37 INA193, U38 INA826, U39 INA193, U4 EG2131, U40 INA826, U41 INA193, U42 INA826, U43 USBLC6-4SC6, U5 EG2131, U6 SN74LVC1G07QDCKTQ1, U7 EG2131, U8 EG2131, U9 ADC081S021CISD/NOPB, Y1 12MHz, Y2 12MHz, Y3 16MHz

Commit message: Latest layout updates, with minor schematic changes.
Parts:
- added C121: 1u, Capacitor_SMD:C_0603_1608Metric, F.Cu at (103.6, 45.5)
- added C122: 1u, Capacitor_SMD:C_0603_1608Metric, F.Cu at (103.5, 37.3)
- added R113: 2mΩ, Resistor_SMD:R_2512_6332Metric, F.Cu at (161.6, 39.0)
- added R114: 2mΩ, Resistor_SMD:R_2512_6332Metric, F.Cu at (161.6, 58.0)
- added R115: 2mΩ, Resistor_SMD:R_2512_6332Metric, F.Cu at (161.7, 89.9)
- added R116: 2mΩ, Resistor_SMD:R_2512_6332Metric, F.Cu at (161.7, 69.2)
- added TP22: TestPoint, TestPoint:TestPoint_Keystone_5019_Minature, F.Cu at (82.4, 75.5)
- R101, R105, R109, R50: value 1mΩ -> 2mΩ
- moved G*** 24.5 mm to (141.0, 87.0)
- moved R11 17.5 mm to (186.6, 92.0)
- moved R17 15.9 mm to (181.7, 93.3)
- moved R12 11.3 mm to (183.5, 93.2)
- moved C102 10.5 mm to (156.3, 32.8)
- moved R87 10.5 mm to (153.2, 32.8)
- moved R90 10.2 mm to (155.7, 43.0)
- moved C105 10.2 mm to (158.8, 43.0)
- moved G*** 9.43 mm to (140.1, 62.1)
- moved G*** 9.35 mm to (140.9, 75.1)
- moved R21 9.22 mm to (163.2, 73.2), turned to 0 degrees
- moved R45 8.97 mm to (165.7, 61.0)
- moved C104 8.49 mm to (162.5, 60.9)
- moved R89 8.49 mm to (159.4, 60.9)
- moved D9 5.98 mm to (167.4, 56.7), turned to -90 degrees
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Connections:
- D18 pad 1: /gate_drive/M2A_P -> /gate_drive/M2A_N
- D26 pad 1: /gate_drive/M1C_P -> /gate_drive/M1C_N
- D42 pad 1: /gate_drive/M1A_P -> /gate_drive/M1A_N
- D9 pad 1: /gate_drive/M2C_P -> /gate_drive/M2C_N
- TH1 pad 1: +3V3 -> +3.3VA
- TH2 pad 1: +3V3 -> +3.3VA
- U1 pad 2: /gate_drive/M1C_PWM_H -> M1C_PWM_H
- U1 pad 3: /gate_drive/M1C_PWM_L\ -> M1C_PWM_L\
- U15 pad 11: /power_and_cpu/M1A_PWM_H -> M1A_PWM_H
- U15 pad 12: /power_and_cpu/M1A_PWM_L\ -> M1A_PWM_L\
- U15 pad 13: /power_and_cpu/M2C_PWM_H -> M2C_PWM_H
- U15 pad 14: /power_and_cpu/M2C_PWM_L\ -> M2C_PWM_L\
- U15 pad 15: /power_and_cpu/M2B_PWM_H -> M2B_PWM_H
- U15 pad 16: /power_and_cpu/M2B_PWM_L\ -> M2B_PWM_L\
- U15 pad 17: /power_and_cpu/M2A_PWM_H -> M2A_PWM_H
- U15 pad 18: /power_and_cpu/M2A_PWM_L\ -> M2A_PWM_L\
- U15 pad 30: unconnected-(U15-GPIO19-Pad30) -> Net-(U15-GPIO19)
- U15 pad 6: /power_and_cpu/M1C_PWM_H -> M1C_PWM_H
- U15 pad 7: /power_and_cpu/M1C_PWM_L\ -> M1C_PWM_L\
- U15 pad 8: /power_and_cpu/M1B_PWM_H -> M1B_PWM_H
- U15 pad 9: /power_and_cpu/M1B_PWM_L\ -> M1B_PWM_L\
- U2 pad 2: /gate_drive/M2C_PWM_H -> M2C_PWM_H
- U2 pad 3: /gate_drive/M2C_PWM_L\ -> M2C_PWM_L\
- U4 pad 2: /gate_drive/M1B_PWM_H -> M1B_PWM_H
- U4 pad 3: /gate_drive/M1B_PWM_L\ -> M1B_PWM_L\
- U5 pad 2: /gate_drive/M2B_PWM_H -> M2B_PWM_H
- U5 pad 3: /gate_drive/M2B_PWM_L\ -> M2B_PWM_L\
- U7 pad 2: /gate_drive/M1A_PWM_H -> M1A_PWM_H
- U7 pad 3: /gate_drive/M1A_PWM_L\ -> M1A_PWM_L\
- U8 pad 2: /gate_drive/M2A_PWM_H -> M2A_PWM_H
- U8 pad 3: /gate_drive/M2A_PWM_L\ -> M2A_PWM_L\
Routing:
- net +3.3VA: track 43.8 -> 328.2 mm, vias 2 -> 12
- net GND: track 17.7 -> 163.0 mm, vias 110 -> 243
- net +12V: track 0.00 -> 134.8 mm, vias 0 -> 8
- net /gate_drive/M1C_P: track 0.00 -> 115.1 mm, vias 0 -> 4
- net +3V3: track 3.42 -> 104.4 mm, vias 0 -> 3
- net /power_and_cpu/ADC_CLK: track 0.00 -> 90.3 mm, vias 0 -> 2
- net /power_and_cpu/ADC_DATA: track 0.00 -> 90.2 mm, vias 0 -> 2
- net /power_and_cpu/ADC_CS2: track 0.00 -> 85.3 mm, vias 0 -> 1
- net /power_and_cpu/ADC_CS3: track 0.00 -> 79.6 mm, vias 0 -> 1
- net VMOT: track 0.00 -> 71.1 mm, vias 0 -> 4
- net /power_and_cpu/GPIO25: track 0.00 -> 65.6 mm, vias 0 -> 2
- net /gate_drive/M1C_N: track 0.00 -> 63.0 mm, vias 0 -> 2
- net /power_and_cpu/GPIO24: track 0.00 -> 60.9 mm, vias 0 -> 1
- net /power_and_cpu/SWCLK: track 0.00 -> 57.9 mm, vias 0 -> 2
- net /power_and_cpu/SWD: track 0.00 -> 51.3 mm, vias 0 -> 1
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- added copper zone on F.Cu, net +5V
- added copper zone on F.Cu, net /gate_drive/M1C_N
Other:
- board text removed: "C1"
- board text removed: "C2"

Commit message: initial 100% routing of PCB done with latest updates
Parts:
- removed TP10, TP11, TP13, TP14, TP15, TP16, TP17, TP18, TP19, TP20, TP21, TP23, TP24, TP25, TP26, TP27, TP28, TP29, TP30, TP31, TP32, TP33, TP34, TP35, TP36, TP37, TP38, TP39, TP40, TP41, TP42, TP43, TP44, TP45, TP46, TP47, TP48, TP49, TP50, TP51, TP52, TP53, TP54, TP56, TP59, TP60, TP61, TP63: TestPoint, TestPoint:TestPoint_Pad_D2.0mm
- removed TP4, TP5, TP6, TP7, TP8, TP9: TestPoint, TestPoint:TestPoint_Pad_D3.0mm
- removed U25: NCP1117-5_SOT223, Package_TO_SOT_SMD:SOT-223-3_TabPin2
- moved G*** 48.1 mm to (141.1, 39.0)
- moved G*** 25.2 mm to (138.4, 50.1)
- moved R17 24.0 mm to (157.8, 95.6), turned to 90 degrees
- moved D37 23.9 mm to (70.8, 102.7)
- moved R11 23.4 mm to (165.2, 101.6), turned to -90 degrees
- moved R12 21.6 mm to (163.6, 101.6), turned to -90 degrees
- moved TP22 19.9 mm to (99.8, 66.0)
- moved R66 18.5 mm to (102.7, 93.1), turned to 90 degrees
- moved R9 9.31 mm to (167.6, 110.0), turned to 0 degrees
- moved C22 8.07 mm to (70.3, 87.0), turned to -90 degrees
- moved C1 6.80 mm to (149.9, 95.1)
- moved C55 6.80 mm to (151.5, 95.1)
- moved FB2 6.80 mm to (153.8, 94.3)
- moved J7 6.30 mm to (162.3, 98.0)
- moved R64 6.15 mm to (76.7, 89.6), turned to 180 degrees
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Connections:
- J17 pad 9: (no net) -> GND_ISO
- J2 pad 9: (no net) -> GND_ISO
- JP2 pad 1: /power_and_cpu/CANL0_N -> /power_and_cpu/CAN0_N
- R10 pad 2: /power_and_cpu/GND_REMOTE -> GND_ISO
- R9 pad 1: /power_and_cpu/CANH0_P -> /power_and_cpu/CAN0_P
- SW3 pad 5: /power_and_cpu/CANL0_N -> /power_and_cpu/CAN0_N
Routing:
- net +3V3: track 104.4 -> 557.8 mm, vias 3 -> 31
- net /power_and_cpu//LED_EN: track 0.00 -> 134.1 mm, vias 0 -> 4
- net /power_and_cpu/ID2: track 0.00 -> 125.1 mm, vias 0 -> 6
- net GND_ISO: track 0.00 -> 121.6 mm, vias 0 -> 4
- net /power_and_cpu/ID1: track 0.00 -> 111.1 mm, vias 0 -> 2
- net /power_and_cpu/ID3: track 0.00 -> 107.8 mm, vias 0 -> 2
- net /power_and_cpu/GPIO29_ADC3_2: track 6.21 -> 105.8 mm, vias 0 -> 3
- net GND: track 163.0 -> 259.5 mm, vias 243 -> 281
- net /power_and_cpu/ESTOP: track 0.00 -> 77.3 mm, vias 0 -> 4
- net +5V: track 51.2 -> 128.4 mm, vias 4 -> 6
- net /power_and_cpu/CAN0_N: track 0.00 -> 72.6 mm, vias 0 -> 3
- net VMOT: track 71.1 -> 143.2 mm, vias 4 -> 8
- net /power_and_cpu/SWCLK_2: track 0.00 -> 68.5 mm, vias 0 -> 2
- net VBUS: track 0.00 -> 64.9 mm
- net +5V_ISO: track 0.00 -> 63.8 mm
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Other:
- board text added: "C1"
- board text added: "C2"

Commit message: board updates just before adding test points
Parts:
- removed H5, H9: MountingHole, RP2040_minimal:MountingHole_3.9mm_Plastite_#6
- added TP10: TestPoint, TestPoint:TestPoint_Pad_D2.0mm, B.Cu at (139.9, -21.7)
- added TP11: TestPoint, TestPoint:TestPoint_Pad_D2.0mm, B.Cu at (139.9, -17.6)
- added TP13: TestPoint, TestPoint:TestPoint_Pad_D2.0mm, B.Cu at (139.9, -13.6)
- added TP14: TestPoint, TestPoint:TestPoint_Pad_D2.0mm, B.Cu at (139.9, -9.53)
- added TP15: TestPoint, TestPoint:TestPoint_Pad_D2.0mm, B.Cu at (139.9, -5.47)
- added TP16: TestPoint, TestPoint:TestPoint_Pad_D2.0mm, B.Cu at (139.9, -1.43)
- added TP17: TestPoint, TestPoint:TestPoint_Pad_D2.0mm, B.Cu at (135.9, -21.7)
- added TP18: TestPoint, TestPoint:TestPoint_Pad_D2.0mm, B.Cu at (135.9, -17.6)
- added TP19: TestPoint, TestPoint:TestPoint_Pad_D2.0mm, B.Cu at (135.9, -13.6)
- added TP20: TestPoint, TestPoint:TestPoint_Pad_D2.0mm, B.Cu at (135.9, -9.53)
- added TP21: TestPoint, TestPoint:TestPoint_Pad_D2.0mm, B.Cu at (135.9, -5.47)
- added TP23: TestPoint, TestPoint:TestPoint_Pad_D2.0mm, B.Cu at (135.9, -1.43)
- added TP24: TestPoint, TestPoint:TestPoint_Pad_D2.0mm, B.Cu at (131.8, -21.7)
- added TP25: TestPoint, TestPoint:TestPoint_Pad_D2.0mm, B.Cu at (131.8, -17.6)
- added TP26: TestPoint, TestPoint:TestPoint_Pad_D2.0mm, B.Cu at (131.8, -13.6)
- added TP27: TestPoint, TestPoint:TestPoint_Pad_D2.0mm, B.Cu at (131.8, -9.53)
- added TP28: TestPoint, TestPoint:TestPoint_Pad_D2.0mm, B.Cu at (131.8, -5.47)
- added TP29: TestPoint, TestPoint:TestPoint_Pad_D2.0mm, B.Cu at (131.8, -1.43)
- added TP30: TestPoint, TestPoint:TestPoint_Pad_D2.0mm, B.Cu at (127.8, -21.7)
- added TP31: TestPoint, TestPoint:TestPoint_Pad_D2.0mm, B.Cu at (127.8, -17.6)
- added TP32: TestPoint, TestPoint:TestPoint_Pad_D2.0mm, B.Cu at (127.8, -13.6)
- added TP33: TestPoint, TestPoint:TestPoint_Pad_D2.0mm, B.Cu at (127.8, -9.53)
- added TP34: TestPoint, TestPoint:TestPoint_Pad_D2.0mm, B.Cu at (127.8, -5.47)
- added TP35: TestPoint, TestPoint:TestPoint_Pad_D2.0mm, B.Cu at (127.8, -1.43)
- added TP36: TestPoint, TestPoint:TestPoint_Pad_D2.0mm, B.Cu at (123.7, -21.7)
- added TP37: TestPoint, TestPoint:TestPoint_Pad_D2.0mm, B.Cu at (123.7, -17.6)
- added TP38: TestPoint, TestPoint:TestPoint_Pad_D2.0mm, B.Cu at (123.7, -13.6)
- added TP39: TestPoint, TestPoint:TestPoint_Pad_D2.0mm, B.Cu at (123.7, -9.53)
- added TP4: TestPoint, TestPoint:TestPoint_Pad_D3.0mm, B.Cu at (139.4, 13.4)
- added TP40: TestPoint, TestPoint:TestPoint_Pad_D2.0mm, B.Cu at (123.7, -5.47)
- added TP41: TestPoint, TestPoint:TestPoint_Pad_D2.0mm, B.Cu at (123.7, -1.43)
- added TP42: TestPoint, TestPoint:TestPoint_Pad_D2.0mm, B.Cu at (119.7, -21.7)
- added TP43: TestPoint, TestPoint:TestPoint_Pad_D2.0mm, B.Cu at (119.7, -17.6)
- added TP44: TestPoint, TestPoint:TestPoint_Pad_D2.0mm, B.Cu at (119.7, -13.6)
- added TP45: TestPoint, TestPoint:TestPoint_Pad_D2.0mm, B.Cu at (119.7, -9.53)
- added TP46: TestPoint, TestPoint:TestPoint_Pad_D2.0mm, B.Cu at (119.7, -5.47)
- added TP47: TestPoint, TestPoint:TestPoint_Pad_D2.0mm, B.Cu at (119.7, -1.43)
- added TP48: TestPoint, TestPoint:TestPoint_Pad_D2.0mm, B.Cu at (115.6, -21.7)
- added TP49: TestPoint, TestPoint:TestPoint_Pad_D2.0mm, B.Cu at (115.6, -17.6)
- added TP5: TestPoint, TestPoint:TestPoint_Pad_D3.0mm, B.Cu at (139.4, 18.4)
- added TP50: TestPoint, TestPoint:TestPoint_Pad_D2.0mm, B.Cu at (115.6, -13.6)
- added TP51: TestPoint, TestPoint:TestPoint_Pad_D2.0mm, B.Cu at (115.6, -9.53)
- added TP52: TestPoint, TestPoint:TestPoint_Pad_D2.0mm, B.Cu at (115.6, -5.47)
- added TP53: TestPoint, TestPoint:TestPoint_Pad_D2.0mm, B.Cu at (115.6, -1.43)
- added TP54: TestPoint, TestPoint:TestPoint_Pad_D2.0mm, B.Cu at (111.6, -21.7)
- added TP56: TestPoint, TestPoint:TestPoint_Pad_D2.0mm, B.Cu at (111.6, -17.6)
- added TP59: TestPoint, TestPoint:TestPoint_Pad_D2.0mm, B.Cu at (111.6, -13.6)
- added TP6: TestPoint, TestPoint:TestPoint_Pad_D3.0mm, B.Cu at (134.4, 13.4)
- added TP60: TestPoint, TestPoint:TestPoint_Pad_D2.0mm, B.Cu at (111.6, -9.53)
- added TP61: TestPoint, TestPoint:TestPoint_Pad_D2.0mm, B.Cu at (118.0, 19.9)
- added TP63: TestPoint, TestPoint:TestPoint_Pad_D2.0mm, B.Cu at (109.0, -3.50)
- added TP7: TestPoint, TestPoint:TestPoint_Pad_D3.0mm, B.Cu at (134.4, 18.4)
- added TP8: TestPoint, TestPoint:TestPoint_Pad_D3.0mm, B.Cu at (129.3, 13.4)
- added TP9: TestPoint, TestPoint:TestPoint_Pad_D3.0mm, B.Cu at (129.3, 18.4)
- added U25: NCP1117-5_SOT223, Package_TO_SOT_SMD:SOT-223-3_TabPin2, B.Cu at (137.0, 4.72)
- moved G*** 22.4 mm to (158.9, 47.5)
- moved G*** 22.1 mm to (152.0, 43.9)
- moved G*** 20.6 mm to (138.5, 44.7)
Routing:
- net /power_and_cpu/SPI1_INT: track 47.2 -> 44.9 mm
- net GND: track 259.5 -> 259.4 mm, vias 281 -> 285
