File: gate_drive.kicad_sch (KiCad schematic)
At the start: 220 parts, among them J19 Conn_01x03, J20 Conn_01x03, Q1 Q_PNP_BEC, Q2 Q_PNP_BEC, Q3 Q_PNP_BEC, Q4 Q_PNP_BEC, Q5 Q_PNP_BEC, Q6 Q_PNP_BEC, U1 EG3113, U14 INA240A1D, U2 EG3113, U20 INA240A1D, U21 INA240A1D, U4 EG3113, U44 INA240A1D, U5 EG3113, U7 EG3113, U8 EG3113

Commit message: Latest updates to module based design.
Parts:
- removed AH1, AH2, AL1, AL2, BH1, BH2, BL1, BL2, CH1, CH2, CL1, CL2: MOSFETSO-8, motor:PowerPAK_SO-8_123, symbol Device:Q_NMOS_SGD
- removed C10, C11, C14, C15, C2, C81: 4.7uF 35V, Capacitor_SMD:C_0603_1608Metric, symbol Device:C
- removed C100, C101, C102, C103, C104, C105, C106, C107, C108, C109, C93, C99: C, Capacitor_SMD:C_0603_1608Metric, symbol Device:C
- removed C12, C16, C17, C25, C82, C9: DNP, Capacitor_SMD:C_0603_1608Metric, symbol Device:C
- removed C13, C65, C70, C71, C84, C85: 10uF 35v, Capacitor_SMD:C_0603_1608Metric, symbol Device:C
- removed C26, C3, C4, C5, C6, C7: 100uF 63V solid, Capacitor_THT:CP_Radial_D8.0mm_P3.50mm, symbol Device:C_Polarized
- removed C59, C66, C72, C74: 100n, Capacitor_SMD:C_0603_1608Metric, symbol Device:C
- removed C68, C76, C77, C78, C79, C80: 2.2uF 100V, Capacitor_SMD:C_1206_3216Metric, symbol Device:C
- removed D10, D11, D19, D2, D21, D7: FR107, Diode_SMD:D_SOD-123, symbol Device:D
- removed D12, D13, D14, D15, D16, D17, D20, D22, D23, D24, D5, D6: CDBU0130R-HF, Diode_SMD:D_SOD-523, symbol Device:D
- removed D18, D25, D26, D42, D8, D9: SMAJ51A, Diode_SMD:D_SMA, symbol Diode:SMF54A
- removed J19, J20: Conn_01x03, parts:MT60-F.G.Y, symbol Connector_Generic:Conn_01x03
- removed Q1, Q2, Q3, Q4, Q5, Q6: Q_PNP_BEC, Package_TO_SOT_SMD:SOT-23, symbol Device:Q_PNP_BEC
- removed R1, R18, R19, R20, R22, R26, R3, R30, R31, R34, R35, R37, R38, R39, R6, R7, R8, R82: 0R, Resistor_SMD:R_0603_1608Metric, symbol MotorController:TAYLOR_RESISTOR
- removed R101, R105, R109, R113, R114, R115, R116, R50: 3mΩ, Resistor_SMD:R_2512_6332Metric, symbol MotorController:TAYLOR_RESISTOR
- removed R108, R110, R111, R112, R117, R118, R119, R120, R121, R122, R123, R124, R125, R126, R127, R128, R129, R130: 10k, Resistor_SMD:R_0603_1608Metric, symbol MotorController:TAYLOR_RESISTOR
- removed R131, R132, R133, R134, R135, R136: 40k, Resistor_SMD:R_0603_1608Metric, symbol MotorController:TAYLOR_RESISTOR
- removed R14, R4, R5, R86, R87, R88, R89, R90, R91, R92, R93, R94: R, Resistor_SMD:R_0603_1608Metric, symbol Device:R
- removed R23, R24, R25, R27, R28, R29, R32, R33, R36, R59, R69, R73, R78, R80, R81, R83, R84, R85: 10.2R, Resistor_SMD:R_0603_1608Metric, symbol MotorController:TAYLOR_RESISTOR
- removed TP12, TP55, TP57, TP58, TP62, TP64, TP65, TP66, TP67, TP68, TP69, TP70, TP71, TP72, TP73, TP74, TP75, TP76, TP77, TP78, TP79, TP80, TP81, TP82, TP83, TP84, TP85, TP86, TP87, TP90, TP91, TP92, TP93, TP94: TestPoint, TestPoint:TestPoint_Pad_D1.5mm, symbol Connector:TestPoint
- removed TP4, TP5, TP6, TP7, TP8, TP9: TestPoint, TestPoint:TestPoint_Pad_D3.0mm, symbol Connector:TestPoint
- removed U1, U2, U4, U5, U7, U8: EG3113, Package_SO:SOIC-8_3.9x4.9mm_P1.27mm, symbol MotorBuck:EG2131
- removed U14, U20, U21, U44: INA240A1D, Package_SO:SOIC-8_3.9x4.9mm_P1.27mm, symbol Amplifier_Current:INA240A1D
Other:
- note removed: "(Motor 1, gate phase A, High)"
- note removed: "MOTOR 1"
- note removed: "MOTOR 2"
- note removed: "Note: EG3113 or EG2131 gate drivers may be used."
